File: hw/3020-cnc-upgrade.kicad_pcb (KiCad board)
At the start: 2 copper layers, 100 x 41 mm, 13 parts, among them P1 CONN_01X02, P2 CONN_01X03, P3 CONN_01X08, P4 CONN_01X03, U1 6N136, U3 MCP41010

Commit message: updated
Parts:
- added U2: arduino_pro_micro, Housings_DIP:DIP-24_W15.24mm, F.Cu at (148.9, 109.4)
- moved P4 31.8 mm to (141.0, 113.0)
- moved P1 18.0 mm to (131.9, 112.6), turned to 0 degrees
- moved U1 15.9 mm to (132.8, 93.2)
- moved P2 12.9 mm to (197.2, 106.1)
- moved D1 12.8 mm to (133.2, 105.0)
- moved R1 12.8 mm to (127.2, 104.0)
- moved U3 7.34 mm to (182.9, 98.5)
- moved P3 6.79 mm to (159.2, 113.8)
Connections:
- P3 pad 2: (no net) -> /P3.6
- P3 pad 3: (no net) -> /P5.4
- P3 pad 4: (no net) -> /P5.5
- P3 pad 6: (no net) -> /P3.1/TX
- P3 pad 7: (no net) -> /P3.0/RX
- P3 pad 8: (no net) -> /P3.2
- P4 pad 2: (no net) -> /POT
- U1 pad 7: (no net) -> Net-(U1-Pad7)
- U3 pad 1: (no net) -> Net-(U2-Pad13)
- U3 pad 2: (no net) -> /SCK
- U3 pad 3: (no net) -> /MOSI
Other:
- outline, holes or cut-outs redrawn

Commit message: pcb layout
Parts:
- moved REF** 32.0 mm to (184.0, 93.0)
- moved REF** 30.1 mm to (184.0, 114.0)
- moved P2 26.3 mm to (172.0, 113.5), turned to 0 degrees
- moved R2 25.5 mm to (135.0, 94.0)
- moved P1 13.1 mm to (125.0, 101.5), turned to 270 degrees
- moved P3 12.7 mm to (146.5, 113.5)
- moved D1 11.1 mm to (132.0, 94.0)
- moved REF** 11.0 mm to (123.0, 93.0)
- moved R1 9.46 mm to (129.0, 94.8), turned to 270 degrees
- moved P4 7.06 mm to (134.0, 113.5)
- moved U2 6.60 mm to (142.8, 107.0)
- moved U1 6.50 mm to (130.2, 99.2)
- moved REF** 2.24 mm to (123.0, 114.0)
- moved U3 1.51 mm to (184.1, 99.4), turned to 270 degrees
Connections:
- net Net-(U2-Pad13) renamed /~CS
- P3 pad 2: /P3.6 -> (no net)
- P3 pad 3: /P5.4 -> (no net)
- P3 pad 4: /P5.5 -> (no net)
- P3 pad 6: /P3.1/TX -> (no net)
- P3 pad 7: /P3.0/RX -> (no net)
- P3 pad 8: /P3.2 -> (no net)
- U1 pad 7: Net-(U1-Pad7) -> (no net)
- U2 pad 1: Net-(U2-Pad1) -> (no net)
- U2 pad 10: Net-(U2-Pad10) -> (no net)
- U2 pad 11: Net-(U2-Pad11) -> (no net)
- U2 pad 12: Net-(U2-Pad12) -> (no net)
- U2 pad 15: /MISO -> (no net)
- U2 pad 18: Net-(U2-Pad18) -> (no net)
- U2 pad 19: Net-(U2-Pad19) -> (no net)
- U2 pad 2: Net-(U2-Pad2) -> (no net)
- U2 pad 20: Net-(U2-Pad20) -> (no net)
- U2 pad 22: Net-(U2-Pad22) -> (no net)
- U2 pad 24: Net-(U2-Pad24) -> (no net)
- U2 pad 6: Net-(U2-Pad6) -> (no net)
- U2 pad 7: Net-(U2-Pad7) -> (no net)
- U2 pad 8: Net-(U2-Pad8) -> (no net)
- U2 pad 9: Net-(U2-Pad9) -> (no net)
Routing:
- net /POT: track 0.00 -> 38.5 mm
- net Net-(R2-Pad2): track 0.00 -> 26.7 mm
- net /SCK: track 0.00 -> 22.6 mm
- net /~CS: track 0.00 -> 16.5 mm
- net Net-(D1-Pad2): track 0.00 -> 14.7 mm
- net /MOSI: track 0.00 -> 14.0 mm
- net Net-(D1-Pad1): track 0.00 -> 13.3 mm
- net Net-(P2-Pad3): track 0.00 -> 8.38 mm
- net Net-(P2-Pad2): track 0.00 -> 8.36 mm
- net Net-(P2-Pad1): track 0.00 -> 8.35 mm
- net Net-(P1-Pad1): track 0.00 -> 7.63 mm
Other:
- board size 100 x 41 mm -> 69 x 29 mm
- net class pwr added: clearance 0.2, trace_width 0.4, via_dia 0.6, via_drill 0.4
- board text added: "1"
- board text added: "10"
- board text added: "14"
- board text added: "15"
- board text added: "16"
- board text added: "2"
- board text added: "21mm"
- board text added: "3"
- board text added: "4"
- board text added: "5"
- board text added: "6"
- board text added: "61mm"
- board text added: "6N136"
- board text added: "7"
- board text added: "8"
- board text added: "9"
- board text added: "A0"
- board text added: "A1"
- board text added: "A2"
- board text added: "A3"
- board text added: "ARDUINO PRO MICRO"
- board text added: "FP POT"
- board text added: "GND"
- board text added: "MCP41010"
- board text added: "PWM IN"
- board text added: "RAW"
- board text added: "RST"
- board text added: "RXI"
- board text added: "TX0"
- board text added: "VCC"

Commit message: updates to layout
Other:
- board text added: "TO PCB POT IN"
Changed lines of the file:
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@@
     (area 111.585714 86 202.000001 120.000001)
     (thickness 1.6)
-    (drawings 67)
+    (drawings 69)
     (tracks 43)
     (zones 0)
@@
     (tags SOD-123)
     (attr smd)
-    (fp_text reference D1 (at -3 -2 270) (layer F.SilkS)
+    (fp_text reference D1 (at -3.1 0 360) (layer F.SilkS)
       (effects (font (size 1 1) (thickness 0.15)))
     )
@@
     (descr "JST XH series connector, B03B-XH-A, top entry type, through hole")
     (tags "connector jst xh tht top vertical 2.50mm")
-    (fp_text reference P2 (at 2.5 -3.5) (layer F.SilkS)
+    (fp_text reference P2 (at -3.5 0 90) (layer F.SilkS)
       (effects (font (size 1 1) (thickness 0.15)))
     )
@@
     (tags "resistor 0805")
     (attr smd)
-    (fp_text reference R2 (at 0 -2.1 270) (layer F.SilkS)
+    (fp_text reference R2 (at -2.4 0 360) (layer F.SilkS)
       (effects (font (size 1 1) (thickness 0.15)))
     )
@@
     (descr "JST XH series connector, B08B-XH-A, top entry type, through hole")
     (tags "connector jst xh tht top vertical 2.50mm")
-    (fp_text reference P3 (at 8.75 -3.5) (layer F.SilkS)
+    (fp_text reference P3 (at -3.5 0 270) (layer F.SilkS)
       (effects (font (size 1 1) (thickness 0.15)))
     )
@@
     (descr "JST XH series connector, B03B-XH-A, top entry type, through hole")
     (tags "connector jst xh tht top vertical 2.50mm")
-    (fp_text reference P4 (at 2.5 -3.5) (layer F.SilkS)
+    (fp_text reference P4 (at -3.5 -0.06 90) (layer F.SilkS)
       (effects (font (size 1 1) (thickness 0.15)))
     )
@@
     (descr "24-lead dip package, row spacing 15.24 mm (600 mils)")
     (tags "dil dip 2.54 600")
-    (fp_text reference U2 (at 0 -5.22 90) (layer F.SilkS)
+    (fp_text reference U2 (at 10.89 -5.76 360) (layer F.SilkS)
       (effects (font (size 1 1) (thickness 0.15)))
     )
@@
     )
   )
+  (gr_text "TO PCB POT IN" (at 174.5 109.7) (layer F.SilkS)
+    (effects (font (size 1 1) (thickness 0.25)))
+  )
+  (gr_text 1 (at 185.8 98.7) (layer F.SilkS)
+    (effects (font (size 1 1) (thickness 0.25)))
+  )
   (gr_line (start 120.5 106.5) (end 120.8 106.2) (layer F.SilkS) (width 0.2))
   (gr_line (start 120.5 106.5) (end 120.2 106.2) (layer F.SilkS) (width 0.2))
@@
     (effects (font (size 1 1) (thickness 0.25)))
   )
-  (gr_text 1 (at 185.928 98.552) (layer F.SilkS)
+  (gr_text 1 (at 129.8 97.3) (layer F.SilkS)
     (effects (font (size 1 1) (thickness 0.25)))
   )
@@
     (effects (font (size 1 1) (thickness 0.25)))
   )
-  (gr_text "FP POT" (at 130 114 90) (layer F.SilkS)
-    (effects (font (size 1 1) (thickness 0.25)))
-  )
+  (gr_text "FP POT" (at 137.4 110.3 360) (layer F.SilkS)
+    (effects (font (size 1 1) (thickness 0.25)))
+  )

Commit message: minor updates to hw
Connections:
- P3 pad 2: (no net) -> /P3.6
- P3 pad 3: (no net) -> /P5.4
- P3 pad 4: (no net) -> /P5.5
- P3 pad 6: (no net) -> /P3.1/TX
- P3 pad 7: (no net) -> /P3.0/RX
- P3 pad 8: (no net) -> /P3.2
- P4 pad 1: +5V -> GND
- P4 pad 3: GND -> +5V
- U1 pad 1: (no net) -> Net-(U1-Pad1)
- U1 pad 4: (no net) -> Net-(U1-Pad4)
- U1 pad 7: (no net) -> Net-(U1-Pad7)
- U2 pad 1: (no net) -> Net-(U2-Pad1)
- U2 pad 10: (no net) -> Net-(U2-Pad10)
- U2 pad 11: (no net) -> Net-(U2-Pad11)
- U2 pad 12: (no net) -> Net-(U2-Pad12)
- U2 pad 15: (no net) -> /MISO
- U2 pad 18: (no net) -> Net-(U2-Pad18)
- U2 pad 19: (no net) -> Net-(U2-Pad19)
- U2 pad 2: (no net) -> Net-(U2-Pad2)
- U2 pad 20: (no net) -> Net-(U2-Pad20)
- U2 pad 22: (no net) -> Net-(U2-Pad22)
- U2 pad 24: (no net) -> Net-(U2-Pad24)
- U2 pad 6: (no net) -> Net-(U2-Pad6)
- U2 pad 7: (no net) -> Net-(U2-Pad7)
- U2 pad 8: (no net) -> Net-(U2-Pad8)
- U2 pad 9: (no net) -> Net-(U2-Pad9)

Commit message: hardware updates
Parts:
- moved P2 7.52 mm to (164.5, 113.0)
- moved P3 4.93 mm to (141.6, 113.0)
- moved P4 2.84 mm to (131.2, 113.0)
Connections:
- P3 pad 1: +5V -> /P3.2
- P3 pad 2: /P3.6 -> /P3.0/RX
- P3 pad 3: /P5.4 -> /P3.1/TX
- P3 pad 4: /P5.5 -> GND
- P3 pad 5: GND -> /P5.5
- P3 pad 6: /P3.1/TX -> /P5.4
- P3 pad 7: /P3.0/RX -> /P3.6
- P3 pad 8: /P3.2 -> +5V
- U3 pad 5: Net-(P2-Pad1) -> Net-(P2-Pad3)
- U3 pad 7: Net-(P2-Pad3) -> Net-(P2-Pad1)
Routing:
- net /POT: track 38.5 -> 53.8 mm
- net Net-(P2-Pad1): track 8.35 -> 21.2 mm
- net Net-(P2-Pad3): track 8.38 -> 18.3 mm
- net Net-(P2-Pad2): track 8.36 -> 14.5 mm

Commit message: swapped pins on pwm input
Connections:
- P1 pad 1: Net-(P1-Pad1) -> Net-(D1-Pad2)
- P1 pad 2: Net-(D1-Pad2) -> Net-(P1-Pad2)
- R1 pad 2: Net-(P1-Pad1) -> Net-(P1-Pad2)
Routing:
- net Net-(P1-Pad2): track 0.00 -> 12.3 mm
- net Net-(P1-Pad1): track 7.63 -> 0.00 mm
- net Net-(D1-Pad2): track 14.7 -> 15.7 mm

Commit message: added URL and revision to board
Other:
- board text added: "https://github.com/MrSurly/3020-software-spindle-control Tag: hw-rev1"
Changed lines of the file:
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@@
   (general
     (links 25)
-    (no_connects 2)
+    (no_connects 0)
     (area 118.924999 88.924999 188.075001 118.075001)
     (thickness 1.6)
-    (drawings 69)
+    (drawings 70)
     (tracks 61)
     (zones 0)
@@
     (descr "8-lead dip package, row spacing 7.62 mm (300 mils)")
     (tags "dil dip 2.54 300")
-    (fp_text reference U3 (at 0 -5.22 270) (layer F.SilkS)
+    (fp_text reference U3 (at -1.88 9.13 360) (layer F.SilkS)
       (effects (font (size 1 1) (thickness 0.15)))
     )
@@
     (descr "JST XH series connector, B08B-XH-A, top entry type, through hole")
     (tags "connector jst xh tht top vertical 2.50mm")
-    (fp_text reference P3 (at -3.5 0 270) (layer F.SilkS)
+    (fp_text reference P3 (at 2.2 -3.3 180) (layer F.SilkS)
       (effects (font (size 1 1) (thickness 0.15)))
     )
@@
     (descr "JST XH series connector, B03B-XH-A, top entry type, through hole")
     (tags "connector jst xh tht top vertical 2.50mm")
-    (fp_text reference P2 (at 2.5 -3.5) (layer F.SilkS)
+    (fp_text reference P2 (at 2.1 -3.3) (layer F.SilkS)
       (effects (font (size 1 1) (thickness 0.15)))
     )
@@
     )
   )
+  (gr_text "https://github.com/MrSurly/3020-software-spindle-control\nTag: hw-rev1" (at 186 103.3) (layer B.SilkS)
+    (effects (font (size 1 1) (thickness 0.25)) (justify left mirror))
+  )
   (gr_text "TO PCB POT IN" (at 174.5 109.7) (layer F.SilkS)
     (effects (font (size 1 1) (thickness 0.25)))
@@
     (effects (font (size 1 1) (thickness 0.25)))
   )
-  (gr_text "FP POT" (at 137.4 110.3) (layer F.SilkS)
-    (effects (font (size 1 1) (thickness 0.25)))
-  )
-  (gr_line (start 128.1 104.7) (end 127.85 104.7) (layer F.SilkS) (width 0.2))
-  (gr_line (start 127.85 104.7) (end 128.1 104.7) (layer F.SilkS) (width 0.2))
-  (gr_line (start 127.85 104.7) (end 127.85 104.45) (layer F.SilkS) (width 0.2))
-  (gr_line (start 128.35 104.2) (end 127.85 104.7) (layer F.SilkS) (width 0.2))
-  (gr_line (start 127.85 103.95) (end 127.85 103.7) (layer F.SilkS) (width 0.2))
-  (gr_line (start 128.1 103.95) (end 127.85 103.95) (layer F.SilkS) (width 0.2))
-  (gr_line (start 127.85 103.95) (end 128.1 103.95) (layer F.SilkS) (width 0.2))
-  (gr_line (start 128.35 103.45) (end 127.85 103.95) (layer F.SilkS) (width 0.2))
-  (gr_line (start 128.6 102.95) (end 128.6 103.45) (layer F.SilkS) (width 0.2))
-  (gr_line (start 128.1 102.95) (end 129.1 102.95) (layer F.SilkS) (width 0.2))
-  (gr_line (start 128.1 102.45) (end 128.6 102.45) (layer F.SilkS) (width 0.2))
-  (gr_line (start 128.6 102.95) (end 128.1 102.45) (layer F.SilkS) (width 0.2))
-  (gr_line (start 129.1 102.45) (end 128.6 102.95) (layer F.SilkS) (width 0.2))
-  (gr_line (start 128.6 102.45) (end 129.1 102.45) (layer F.SilkS) (width 0.2))
-  (gr_line (start 128.6 101.95) (end 128.6 102.45) (layer F.SilkS) (width 0.2))
+  (gr_text "FP POT" (at 135 109.9) (layer F.SilkS)
+    (effects (font (size 1 1) (thickness 0.25)))
+  )
+  (gr_line (start 128.91999 101.014315) (end 129.169989 101.014314) (layer F.SilkS) (width 0.2))
+  (gr_line (start 129.169989 101.014314) (end 128.91999 101.014315) (layer F.SilkS) (width 0.2))
+  (gr_line (start 129.169989 101.014314) (end 129.169989 101.264314) (layer F.SilkS) (width 0.2))
+  (gr_line (start 128.669989 101.514313) (end 129.169989 101.014314) (layer F.SilkS) (width 0.2))
+  (gr_line (start 129.169989 101.764314) (end 129.169989 102.014314) (layer F.SilkS) (width 0.2))
+  (gr_line (start 128.91999 101.764315) (end 129.169989 101.764314) (layer F.SilkS) (width 0.2))
+  (gr_line (start 129.169989 101.764314) (end 128.91999 101.764315) (layer F.SilkS) (width 0.2))
+  (gr_line (start 128.669988 102.264314) (end 129.169989 101.764314) (layer F.SilkS) (width 0.2))
+  (gr_line (start 128.41999 102.764314) (end 128.41999 102.264315) (layer F.SilkS) (width 0.2))
+  (gr_line (start 128.91999 102.764314) (end 127.919988 102.764315) (layer F.SilkS) (width 0.2))
+  (gr_line (start 128.91999 103.264314) (end 128.419989 103.264314) (layer F.SilkS) (width 0.2))
+  (gr_line (start 128.41999 102.764314) (end 128.91999 103.264314) (layer F.SilkS) (width 0.2))
+  (gr_line (start 127.919989 103.264314) (end 128.41999 102.764314) (layer F.SilkS) (width 0.2))
+  (gr_line (start 128.419989 103.264314) (end 127.919989 103.264314) (layer F.SilkS) (width 0.2))
+  (gr_line (start 128.41999 103.764314) (end 128.419989 103.264314) (layer F.SilkS) (width 0.2))
   (gr_text "PWM IN" (at 124.5 108) (layer F.SilkS)
     (effects (font (size 1 1) (thickness 0.25)))
