File: hw/3020-cnc-upgrade.sch (KiCad schematic (older format))
At the start: 10 parts, among them P1 CONN_01X02, P2 CONN_01X03, P3 CONN_01X08, P4 CONN_01X03, U1 6N136, U2 arduino_pro_micro, U3 MCP41010

Commit message: added jumper to reverse spindle polarity
Parts:
- added J1: CONN_01X02, Pin_Headers:Pin_Header_Straight_1x02_Pitch2.54mm, symbol CONN_01X02
Connections:
- net GND: now also J1.1 (P1)
- net pol: now reaches U2.6 (3)
- net pol: now also J1.2 (P2)
Changed lines of the file:
@@
 Text Label 5825 4475 0    60   ~ 0
 ~CS
+$Comp
+L CONN_01X02 J1
+U 1 1 5ABA669E
+P 2250 2400
+F 0 "J1" H 2250 2550 50  0000 C CNN
+F 1 "CONN_01X02" V 2350 2400 50  0000 C CNN
+F 2 "Pin_Headers:Pin_Header_Straight_1x02_Pitch2.54mm" H 2250 2400 50  0001 C CNN
+F 3 "" H 2250 2400 50  0001 C CNN
+	1    2250 2400
+	0    -1   -1   0
+$EndComp
+$Comp
+L GND #PWR05
+U 1 1 5ABA677C
+P 2200 2700
+F 0 "#PWR05" H 2200 2450 50  0001 C CNN
+F 1 "GND" H 2200 2550 50  0000 C CNN
+F 2 "" H 2200 2700 50  0000 C CNN
+F 3 "" H 2200 2700 50  0000 C CNN
+	1    2200 2700
+	1    0    0    -1
+$EndComp
+Wire Wire Line
+	2200 2700 2200 2600
+Wire Wire Line
+	2300 2600 2300 2700
+Wire Wire Line
+	2300 2700 3025 2700
+Text Label 3025 2700 2    60   ~ 0
+pol
+Wire Wire Line
+	4825 3875 4275 3875
+Text Label 4275 3875 0    60   ~ 0
+pol
 $EndSCHEMATC

Commit message: added jumper to reverse spindle polarity
Other:
- note added: "PWM polarity\nopen = postitive PWM\n"
Changed lines of the file:
@@
 Text Label 4275 3875 0    60   ~ 0
 pol
+Text Notes 2025 2200 0    60   ~ 0
+PWM polarity\nopen = postitive PWM\n
 $EndSCHEMATC
